File: kicad/PowerSupply_sch.kicad_sch (KiCad schematic)
At the start: 18 parts, among them J1 Jack-DC, SW1 SW_Push_Open, U1 LM7812_TO220, U2 LM7805_TO220, U3 LM7912_TO220

Commit message: Redrawed schematic
Parts:
- renumbered U1 to Q2_I
Connections:
- net +5V: now reaches C8_I.1, U2.3 (VO)
- net +12V: now reaches C6_I.1, Q2_I.3 (VO)
- net -12V: now reaches C7_I1.2, U3.3 (VO)
- no-connect marks 1 -> 0
Other:
- moved on the sheet: C1, C3, C5, C6_I, C7_I1, C8_I, D1, D2, D3, D4, D5, Q2_I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
